Commit message: got links rough drafted:

File: emcee_description/urdf/emcee.urdf.xacro (robot description, xacro)
@@ -13,5 +13,5 @@
   <xacro:property name="chassis_width" value="0.4731"/>
   <xacro:property name="chassis_length" value="0.627"/>
-  <xacro:property name="sled_hoz_width" value="0.44.2"/>
+  <xacro:property name="sled_hoz_width" value="0.442"/>
   <xacro:property name="sled_hoz_length" value="0.245"/>
   <xacro:property name="sled_hoz_height" value="0.0405"/>
@@ -129,5 +129,5 @@
       </geometry>
       <origin xyz="0 0 0" rpy="0 0 0"/>
-      <material name="green"/>
+      <material name="light_grey"/>
     </visual>
     <collision>
@@ -149,6 +149,6 @@
     <!-- <dynamics damping="0.1" friction="0"/> -->
     <dynamics damping="100" friction="1"/>
-    <limit effort="1000" lower="${-(chassis_length/2)-0.0508+(sled_hoz_width/2)}" upper="${(chassis_length/2)-0.0508-(sled_hoz_width/2)}" velocity="0.1"/>
-    <origin rpy="0 0 0" xyz="0 0 ${(chassis_height/2)+0.04}"/>
+    <limit effort="1000" lower="${-(chassis_length/2)+(sled_hoz_width/2)}" upper="${(chassis_length/2)-(sled_hoz_width/2)}" velocity="0.1"/>
+    <origin rpy="0 0 0" xyz="0 0 ${(chassis_height/2)}"/>
   </joint>
   <link name="sled_ver">
@@ -158,5 +158,5 @@
       </geometry>
       <origin xyz="0 0 0" rpy="0 0 0"/>
-      <material name="green"/>
+      <material name="light_grey"/>
     </visual>
     <collision>
@@ -199,5 +199,5 @@
     <parent link="sled_ver"/>
     <child link="arm_s"/>
-    <origin xyz="-0.236 0 ${arm_block_height + 0.0255}"/>
+    <origin xyz="0 0 0"/>
     <axis xyz="0 1 0"/>
     <limit lower="-0.253177" upper="0.30918" effort="1000000" velocity="0.1"/>

Commit message: changed order of lwh

File: emcee_description/urdf/emcee.urdf.xacro (robot description, xacro)
@@ -126,5 +126,5 @@
     <visual>
       <geometry>
-        <box size="${sled_hoz_width} ${sled_hoz_length} ${sled_hoz_height}"/>
+        <box size="${sled_hoz_length} ${sled_hoz_width} ${sled_hoz_height}"/>
       </geometry>
       <origin xyz="0 0 0" rpy="0 0 0"/>
@@ -134,5 +134,5 @@
       <origin xyz="0 0 0"/>
       <geometry>
-        <box size="${sled_hoz_width} ${sled_hoz_length} ${sled_hoz_height}"/>
+        <box size="${sled_hoz_length} ${sled_hoz_width} ${sled_hoz_height}"/>
       </geometry>
     </collision>
@@ -155,5 +155,5 @@
     <visual>
       <geometry>
-        <box size="${sled_ver_width} ${sled_ver_length} ${sled_ver_height}"/>
+        <box size="${sled_ver_length} ${sled_ver_width} ${sled_ver_height}"/>
       </geometry>
       <origin xyz="0 0 0" rpy="0 0 0"/>
@@ -163,5 +163,5 @@
       <origin xyz="0 0 0"/>
       <geometry>
-        <box size="${sled_ver_width} ${sled_ver_length} ${sled_ver_height}"/>
+        <box size="${sled_ver_length} ${sled_ver_width} ${sled_ver_height}"/>
       </geometry>
     </collision>

Commit message: changed order of lwh

File: emcee_description/urdf/emcee.urdf.xacro (robot description, xacro)
@@ -181,5 +181,5 @@
      <origin xyz="0 0 0"/>
       <geometry>
-        <box size="${arm_s_width} ${arm_s_height} ${arm_s_height}"/>
+        <box size="${arm_s_length} ${arm_s_width} ${arm_s_height}"/>
       </geometry>
     </visual>
@@ -187,5 +187,5 @@
       <origin xyz="0.01 -.01 .02"/>
       <geometry>
-        <box size="${arm_s_width} ${arm_s_height} ${arm_s_height}"/>
+        <box size="${arm_s_length} ${arm_s_width} ${arm_s_height}"/>
       </geometry>
     </collision>
@@ -208,5 +208,5 @@
      <origin xyz="0 0 0"/>
       <geometry>
-        <box size="${arm_b_width} ${arm_b_height} ${arm_b_height}"/>
+        <box size="${arm_b_length} ${arm_b_width} ${arm_b_height}"/>
       </geometry>
     </visual>
@@ -214,5 +214,5 @@
       <origin xyz="0.01 -.01 .02"/>
       <geometry>
-        <box size="${arm_b_width} ${arm_b_height} ${arm_b_height}"/>
+        <box size="${arm_b_length} ${arm_b_width} ${arm_b_height}"/>
       </geometry>
     </collision>

Commit message: adjusted all link configurations. new bucket needs to be imported

File: emcee_description/urdf/emcee.urdf.xacro (robot description, xacro)
@@ -23,12 +23,13 @@
   <xacro:property name="arm_s_height" value="0.0405"/>
   <xacro:property name="arm_angle" value="2.356194490192345"/> <!-- 135 degrees -->
-  <xacro:property name="arm_b_width" value="0.350"/>
+  <xacro:property name="arm_b_width" value="0.429"/>
   <xacro:property name="arm_b_length" value="0.440"/>
   <xacro:property name="arm_b_height" value="0.0405"/>
   <!-- TODO: measure these -->
-  <xacro:property name="wheel_radius" value="0.156369"/>
-  <xacro:property name="wheel_width" value="0.1905"/>
-  <xacro:property name="wheel_location_from_back" value="0.2572"/>
-  <xacro:property name="wheel_location_from_front" value="0.08255"/>
+  <xacro:property name="wheel_base" value="0.503"/>
+  <xacro:property name="wheel_track" value="0.575"/>
+  <xacro:property name="wheel_radius" value="0.14"/>
+  <xacro:property name="wheel_width" value="0.17"/>
+  <!-- not sure about this one -->
   <xacro:property name="wheel_height" value="0.047625"/>
   <xacro:macro name="wheel" params="prefix reflect *joint_pose">
@@ -112,14 +113,14 @@
   </link>
   <xacro:wheel prefix="left_front" reflect="1">
-    <origin xyz="${(chassis_length/2)-(wheel_location_from_front)} ${(chassis_width/2)+(wheel_width/2)} ${-(chassis_height/2)+wheel_height}" rpy="0 0 0"/>
+    <origin xyz="${wheel_base/2} ${wheel_track/2} 0" rpy="0 0 0"/>
   </xacro:wheel>
   <xacro:wheel prefix="left_rear" reflect="1">
-    <origin xyz="${-(chassis_length/2)+(wheel_location_from_back)} ${(chassis_width/2)+(wheel_width/2)} ${-(chassis_height/2)+wheel_height}" rpy="0 0 0"/>
+      <origin xyz="${-wheel_base/2} ${wheel_track/2} 0" rpy="0 0 0"/>
   </xacro:wheel>
   <xacro:wheel prefix="right_front" reflect="-1">
-    <origin xyz="${(chassis_length/2)-(wheel_location_from_front)} ${-(chassis_width/2)-(wheel_width/2)} ${-(chassis_height/2)+wheel_height}" rpy="${PI} 0 0"/>
+      <origin xyz="${wheel_base/2} ${-wheel_track/2} 0" rpy="0 0 0"/>
   </xacro:wheel>
   <xacro:wheel prefix="right_rear" reflect="-1">
-    <origin xyz="${-(chassis_length/2)+(wheel_location_from_back)} ${-(chassis_width/2)-(wheel_width/2)} ${-(chassis_height/2)+wheel_height}" rpy="${PI} 0 0"/>
+    <origin xyz="${-wheel_base/2} ${-wheel_track/2} 0" rpy="${PI} 0 0"/>
   </xacro:wheel>
   <link name="sled_hoz">
@@ -149,6 +150,6 @@
     <!-- <dynamics damping="0.1" friction="0"/> -->
     <dynamics damping="100" friction="1"/>
-    <limit effort="1000" lower="${-(chassis_length/2)+(sled_hoz_width/2)}" upper="${(chassis_length/2)-(sled_hoz_width/2)}" velocity="0.1"/>
-    <origin rpy="0 0 0" xyz="0 0 ${(chassis_height/2)}"/>
+    <limit effort="1000" lower="${-(chassis_length/2)+(sled_hoz_length/2)}" upper="${(chassis_length/2)-(sled_hoz_length/2)}" velocity="0.1"/>
+    <origin rpy="0 0 0" xyz="0 0 ${chassis_height/2 + sled_hoz_height/2}"/>
   </joint>
   <link name="sled_ver">
@@ -172,12 +173,12 @@
     </inertial>
   </link>
-  <joint name="sled_bend_joint" type="fixed">
+  <joint name="sled_ver_joint" type="fixed">
     <parent link="sled_hoz"/>
     <child link="sled_ver"/>
-    <origin rpy="0 0 0" xyz="0 0 ${sled_hoz_height}"/>
+    <origin rpy="0 0 0" xyz="${-sled_hoz_length/2 + sled_ver_length/2} 0 ${sled_ver_height/2 + sled_hoz_height/2}"/>
   </joint>
   <link name="arm_s">
     <visual>
-     <origin xyz="0 0 0"/>
+     <origin xyz="${arm_s_length/2 - sled_ver_length/2} 0 0"/>
       <geometry>
         <box size="${arm_s_length} ${arm_s_width} ${arm_s_height}"/>
@@ -185,5 +186,5 @@
     </visual>
     <collision>
-      <origin xyz="0.01 -.01 .02"/>
+      <origin xyz="${arm_s_length/2 - sled_ver_length/2} 0 0"/>
       <geometry>
         <box size="${arm_s_length} ${arm_s_width} ${arm_s_height}"/>
@@ -196,8 +197,8 @@
     </inertial>
   </link>
-  <joint name="arm_joint" type="revolute">
+  <joint name="arm_s_joint" type="revolute">
     <parent link="sled_ver"/>
     <child link="arm_s"/>
-    <origin xyz="0 0 0"/>
+    <origin xyz="0 0 ${sled_ver_height/2}"/>
     <axis xyz="0 1 0"/>
     <limit lower="-0.253177" upper="0.30918" effort="1000000" velocity="0.1"/>
@@ -212,5 +213,5 @@
     </visual>
     <collision>
-      <origin xyz="0.01 -.01 .02"/>
+      <origin xyz="0 0 0"/>
       <geometry>
         <box size="${arm_b_length} ${arm_b_width} ${arm_b_height}"/>
@@ -226,5 +227,5 @@
     <parent link="arm_s"/>
     <child link="arm_b"/>
-    <origin xyz="0 0 0"/>
+    <origin xyz="${arm_s_length/2 + arm_b_length/sqrt(2) + sled_ver_length} 0 ${-arm_b_length/sqrt(2)/2}" rpy="0 ${PI - arm_angle} 0"/>
   </joint>
 <link name="bucket">
@@ -245,5 +246,5 @@
       <!-- xyz="-0.304153 0.030822 -0.01735" -->
       <!-- <origin xyz="0.1 0 0.05" rpy="0 0 0"/> -->
-      <origin xyz="0.124844 -0.000416 0.002654" rpy="0 ${PI/7} 0"/>
+      <origin xyz="0 0 0" rpy="0 ${PI/7} 0"/>
       <!-- <mass value="1"/> -->
       <mass value="3.92566"/>
@@ -255,5 +256,6 @@
     <child link="bucket"/>
     <axis xyz="0 1 0"/>
-    <origin xyz=".965 0 -0.282"/>
+    <!-- <origin xyz="${arm_b_length/sqrt(2)} 0 ${-arm_b_length/sqrt(2)}"/> -->
+    <origin xyz="${arm_b_length/sqrt(2)} 0 0"/>
     <limit lower="${-0.40}" upper="${3.14159/2}" effort="100000" velocity="1"/>
     <dynamics damping="0.1" friction="0"/>
@@ -282,9 +284,4 @@
     <origin rpy="0 0 0" xyz="0.015 0 .07"/>
   </joint>
-  <!-- TODO: This is the note from the copy and paste:
-       Make this internal_imu_link or something, and use a mixed-in xacro
-       to supply the joint between it and imu_link. This is important so that imu_link
-       always points to the "active" IMU. When an upgrade IMU is connected, the
-       internal_imu_link should remain, but imu_link should point to the upgrade one. -->
   <link name="imu_link">
     <inertial>
@@ -298,5 +295,5 @@
     <child link="imu_link"/>
   </joint>
-  <!-- Bring in simulation data for Gazebo. -->
+  <!-- Bring in simulation configuration for Gazebo. -->
   <xacro:include filename="emcee.gazebo"/>
   <transmission name="sled_hoz_trans">

Commit message: added controller stuff

File: emcee_description/urdf/emcee.urdf.xacro (robot description, xacro)
@@ -119,5 +119,5 @@
   </xacro:wheel>
   <xacro:wheel prefix="right_front" reflect="-1">
-      <origin xyz="${wheel_base/2} ${-wheel_track/2} 0" rpy="0 0 0"/>
+      <origin xyz="${wheel_base/2} ${-wheel_track/2} 0" rpy="${PI} 0 0"/>
   </xacro:wheel>
   <xacro:wheel prefix="right_rear" reflect="-1">
@@ -184,4 +184,5 @@
         <box size="${arm_s_length} ${arm_s_width} ${arm_s_height}"/>
       </geometry>
+      <material name="red"/>
     </visual>
     <collision>
@@ -190,4 +191,5 @@
         <box size="${arm_s_length} ${arm_s_width} ${arm_s_height}"/>
       </geometry>
+      <material name="red"/>
     </collision>
     <inertial>
@@ -211,4 +213,5 @@
         <box size="${arm_b_length} ${arm_b_width} ${arm_b_height}"/>
       </geometry>
+      <material name="red"/>
     </visual>
     <collision>
@@ -217,4 +220,5 @@
         <box size="${arm_b_length} ${arm_b_width} ${arm_b_height}"/>
       </geometry>
+      <material name="red"/>
     </collision>
     <inertial>
@@ -309,5 +313,5 @@
   <transmission name="arm_trans">
     <type>transmission_interface/SimpleTransmission</type>
-    <joint name="arm_joint">
+    <joint name="arm_s_joint">
       <hardwareInterface>EffortJointInterface</hardwareInterface>
     </joint>

Commit message: finished new urdf with inertia

File: emcee_description/urdf/emcee.urdf.xacro (robot description, xacro)
@@ -10,4 +10,5 @@
   <material name="black"><color rgba="0.15 0.15 0.15 1.0"/></material>
   <material name="green"><color rgba="0 1 0 1"/></material>
+  <material name="invisible"><color rgba="0 0 0 0"/></material>
   <xacro:property name="chassis_height" value="0.136"/>
   <xacro:property name="chassis_width" value="0.4731"/>
@@ -19,11 +20,11 @@
   <xacro:property name="sled_ver_length" value="0.0405"/>
   <xacro:property name="sled_ver_height" value="0.425"/>
-  <xacro:property name="arm_s_width" value="0.429"/>
-  <xacro:property name="arm_s_length" value="0.452"/>
-  <xacro:property name="arm_s_height" value="0.0405"/>
+  <xacro:property name="arm_upper_width" value="0.429"/>
+  <xacro:property name="arm_upper_length" value="0.452"/>
+  <xacro:property name="arm_upper_height" value="0.0405"/>
   <xacro:property name="arm_angle" value="2.356194490192345"/> <!-- 135 degrees -->
-  <xacro:property name="arm_b_width" value="0.429"/>
-  <xacro:property name="arm_b_length" value="0.440"/>
-  <xacro:property name="arm_b_height" value="0.0405"/>
+  <xacro:property name="arm_lower_width" value="0.429"/>
+  <xacro:property name="arm_lower_length" value="0.440"/>
+  <xacro:property name="arm_lower_height" value="0.0405"/>
   <!-- TODO: measure these -->
   <xacro:property name="wheel_base" value="0.503"/>
@@ -94,20 +95,18 @@
       <origin xyz="0 0 0"/>
       <geometry>
+          <mesh filename="package://emcee_description/meshes/visual/chassis.dae"/>
+      </geometry>
+      <material name="red"/>
+    </visual>
+    <collision>
+      <origin xyz="0 0 0"/>
+      <geometry>
         <box size="${chassis_length} ${chassis_width} ${chassis_height}"/>
       </geometry>
-      <material name="red"/>
-    </visual>
-    <collision>
-      <origin xyz="0 0 0"/>
-      <geometry>
-        <box size="${chassis_length} ${chassis_width} ${chassis_height}"/>
-      </geometry>
-    </collision>
-    <inertial>
-      <origin xyz="0 0 0" rpy="0 0 0"/>
-      <!-- <origin xyz="0.39809 0.40556 0.64213" rpy="0 0 0" /> -->
-      <!-- <mass value="1" /> -->
-      <mass value="18.65"/>
-      <inertia ixx="0.541922" ixy="2.8e-5" ixz="-0.01424" iyy="1.50291" iyz="0.000144" izz="1.71709"/>
+    </collision>
+    <inertial>
+      <origin xyz="0 0 0" rpy="0 0 0"/>
+      <mass value="3.05"/>
+      <inertia ixx="0.28" ixy="0.00" ixz="0.00" iyy="0.42" iyz="0.00" izz="0.17"/>
     </inertial>
   </link>
@@ -127,22 +126,23 @@
     <visual>
       <geometry>
+          <mesh filename="package://emcee_description/meshes/visual/sled.dae"/>
+      </geometry>
+      <origin xyz="0 0 0" rpy="0 0 0"/>
+      <material name="light_grey"/>
+    </visual>
+    <collision>
+      <origin xyz="0 0 0"/>
+      <geometry>
         <box size="${sled_hoz_length} ${sled_hoz_width} ${sled_hoz_height}"/>
       </geometry>
-      <origin xyz="0 0 0" rpy="0 0 0"/>
-      <material name="light_grey"/>
-    </visual>
-    <collision>
-      <origin xyz="0 0 0"/>
-      <geometry>
-        <box size="${sled_hoz_length} ${sled_hoz_width} ${sled_hoz_height}"/>
-      </geometry>
-    </collision>
-    <inertial>
-      <origin xyz="0 0 0" rpy="0 0 0"/>
-      <mass value="12.25"/>
-      <inertia ixx="0.225942" ixy="-5.6e-5" ixz="0.041831" iyy="0.162776" iyz="4.5e-5" izz="0.312502"/>
-    </inertial>
-  </link>
-  <joint name="sled_hoz_joint" type="prismatic">
+    </collision>
+    <inertial>
+      <origin xyz="0 0 0" rpy="0 0 0"/>
+      <mass value="3.0"/>
+      <!-- izz="-0.28" iyy="1.00" iyz="-0.96" ixx="0.96" ixy="0. -->
+    <inertia ixx="0.08" ixy="0.00" ixz="-0.01" iyy="0.06" iyz="0.00" izz="0.04"/>
+    </inertial>
+  </link>
+  <joint name="sled_joint" type="prismatic">
     <parent link="chassis"/>
     <child link="sled_hoz"/>
@@ -156,8 +156,9 @@
     <visual>
       <geometry>
-        <box size="${sled_ver_length} ${sled_ver_width} ${sled_ver_height}"/>
-      </geometry>
-      <origin xyz="0 0 0" rpy="0 0 0"/>
-      <material name="light_grey"/>
+        <!-- <box size="${sled_ver_length} ${sled_ver_width} ${sled_ver_height}"/> -->
+        <box size="0.001 0.001 0.001"/>
+      </geometry>
+      <origin xyz="0 0 0" rpy="0 0 0"/>
+      <material name="invisible"/>
     </visual>
     <collision>
@@ -178,62 +179,64 @@
     <origin rpy="0 0 0" xyz="${-sled_hoz_length/2 + sled_ver_length/2} 0 ${sled_ver_height/2 + sled_hoz_height/2}"/>
   </joint>
-  <link name="arm_s">
-    <visual>
-     <origin xyz="${arm_s_length/2 - sled_ver_length/2} 0 0"/>
-      <geometry>
-        <box size="${arm_s_length} ${arm_s_width} ${arm_s_height}"/>
+  <link name="arm_upper">
+    <visual>
+     <origin xyz="${arm_upper_length/2 - sled_ver_length/2} 0 0"/>
+      <geometry>
+          <mesh filename="package://emcee_description/meshes/visual/arms.dae"/>
       </geometry>
       <material name="red"/>
     </visual>
     <collision>
-      <origin xyz="${arm_s_length/2 - sled_ver_length/2} 0 0"/>
-      <geometry>
-        <box size="${arm_s_length} ${arm_s_width} ${arm_s_height}"/>
+      <origin xyz="${arm_upper_length/2 - sled_ver_length/2} 0 0"/>
+      <geometry>
+        <box size="${arm_upper_length} ${arm_upper_width} ${arm_upper_height}"/>
       </geometry>
       <material name="red"/>
     </collision>
     <inertial>
-      <origin xyz="0.439315 0.004673 -0.035609" rpy="0 0 0"/>
-      <mass value="6.14067"/>
-      <inertia iyy="0.581471" ixy="6.6e-5" iyz="-3e-6" ixx="0.39687" ixz="-0.128097" izz="0.87075"/>
-    </inertial>
-  </link>
-  <joint name="arm_s_joint" type="revolute">
+      <origin xyz="0 0 0" rpy="0 0 0"/>
+      <mass value="2.5"/>
+      <inertia ixx="0.04" ixz="-0.02" ixy="0.00" izz="0.07" iyz="0.0" iyy="0.05" />
+      <!-- <inertia ixx="0.93" ixy="0.00" ixz="-0.37" iyy="-1.00" izz="0.93" /> -->
+    </inertial>
+  </link>
+  <joint name="arm_joint" type="revolute">
     <parent link="sled_ver"/>
-    <child link="arm_s"/>
+    <child link="arm_upper"/>
     <origin xyz="0 0 ${sled_ver_height/2}"/>
     <axis xyz="0 1 0"/>
-    <limit lower="-0.253177" upper="0.30918" effort="1000000" velocity="0.1"/>
+    <limit lower="-0.8" upper="0.31" effort="1000000" velocity="0.1"/>
     <dynamics damping="0.1" friction="0"/>
   </joint>
-  <link name="arm_b">
+  <link name="arm_lower">
     <visual>
      <origin xyz="0 0 0"/>
       <geometry>
-        <box size="${arm_b_length} ${arm_b_width} ${arm_b_height}"/>
+        <!-- <box size="${arm_lower_length} ${arm_lower_width} ${arm_lower_height}"/> -->
+        <box size="0.001 0.001 0.001"/>
+      </geometry>
+      <material name="invisible"/>
+    </visual>
+    <collision>
+      <origin xyz="0 0 0"/>
+      <geometry>
+        <box size="${arm_lower_length} ${arm_lower_width} ${arm_lower_height}"/>
       </geometry>
       <material name="red"/>
-    </visual>
-    <collision>
-      <origin xyz="0 0 0"/>
-      <geometry>
-        <box size="${arm_b_length} ${arm_b_width} ${arm_b_height}"/>
-      </geometry>
-      <material name="red"/>
     </collision>
     <inertial>
       <origin xyz="0.439315 0.004673 -0.035609" rpy="0 0 0"/>
-      <mass value="6.14067"/>
-      <inertia iyy="0.581471" ixy="6.6e-5" iyz="-3e-6" ixx="0.39687" ixz="-0.128097" izz="0.87075"/>
-    </inertial>
-  </link>
-  <joint name="arm_bend_joint" type="fixed">
-    <parent link="arm_s"/>
-    <child link="arm_b"/>
-    <origin xyz="${arm_s_length/2 + arm_b_length/sqrt(2) + sled_ver_length} 0 ${-arm_b_length/sqrt(2)/2}" rpy="0 ${PI - arm_angle} 0"/>
+      <mass value="0.0"/>
+      <inertia ixx="${dummy_inertia}" ixy="0" ixz="0" iyy="${dummy_inertia}" iyz="0" izz="${dummy_inertia}" />
+    </inertial>
+  </link>
+  <joint name="arm_lower_joint" type="fixed">
+    <parent link="arm_upper"/>
+    <child link="arm_lower"/>
+    <origin xyz="${arm_upper_length/2 + arm_lower_length/sqrt(2) + sled_ver_length} 0 ${-arm_lower_length/sqrt(2)/2}" rpy="0 ${PI - arm_angle} 0"/>
   </joint>
 <link name="bucket">
     <visual>
-      <origin xyz="0.00 0 0.00"/>
+      <origin xyz="0.09 0 0.0"/>
       <geometry>
         <mesh filename="package://emcee_description/meshes/visual/bucket.dae"/>
@@ -242,25 +245,21 @@
     </visual>
     <collision>
-      <origin xyz="0.00 0 0.00"/>
-      <geometry>
-        <mesh filename="package://emcee_description/meshes/collision/bucket_simple.dae"/>
-      </geometry>
-    </collision>
-    <inertial>
-      <!-- xyz="-0.304153 0.030822 -0.01735" -->
-      <!-- <origin xyz="0.1 0 0.05" rpy="0 0 0"/> -->
-      <origin xyz="0 0 0" rpy="0 ${PI/7} 0"/>
-      <!-- <mass value="1"/> -->
-      <mass value="3.92566"/>
-      <inertia ixx="0.216901" ixy="0" ixz="-0.007835" iyy="0.042509" iyz="0" izz="0.243738"/>
+      <origin xyz="0.09 0 0.0"/>
+      <geometry>
+          <mesh filename="package://emcee_description/meshes/visual/bucket.dae"/>
+      </geometry>
+    </collision>
+    <inertial>
+      <origin xyz="0 0 0" rpy="0 0 0"/>
+      <mass value="2.45"/>
+      <inertia ixx="0.19" ixy="0.0" ixz="0.00" iyy="0.03" iyz="0.00" izz="0.17"/>
     </inertial>
   </link>
   <joint name="bucket_joint" type="revolute">
-    <parent link="arm_b"/>
+    <parent link="arm_lower"/>
     <child link="bucket"/>
     <axis xyz="0 1 0"/>
-    <!-- <origin xyz="${arm_b_length/sqrt(2)} 0 ${-arm_b_length/sqrt(2)}"/> -->
-    <origin xyz="${arm_b_length/sqrt(2)} 0 0"/>
-    <limit lower="${-0.40}" upper="${3.14159/2}" effort="100000" velocity="1"/>
+    <origin xyz="${arm_lower_length/sqrt(2) - 0.07} 0 -0.03"/>
+    <limit lower="${-1.5}" upper="${0.7}" effort="100000" velocity="1"/>
     <dynamics damping="0.1" friction="0"/>
   </joint>
@@ -283,8 +282,7 @@
   </link>
   <joint name="zed_joint" type="fixed">
-    <parent link="arm_b"/>
+    <parent link="arm_lower"/>
     <child link="zed_link"/>
-    <!-- TODO: get exact position -->
-    <origin rpy="0 0 0" xyz="0.015 0 .07"/>
+    <origin rpy="0 ${-pi/8} 0" xyz="${-arm_lower_length/(1.35*sqrt(2))} 0.0 0.0"/>
   </joint>
   <link name="imu_link">
@@ -303,5 +301,5 @@
   <transmission name="sled_hoz_trans">
     <type>transmission_interface/SimpleTransmission</type>
-    <joint name="sled_hoz_joint">
+    <joint name="sled_joint">
       <hardwareInterface>EffortJointInterface</hardwareInterface>
     </joint>
@@ -313,5 +311,5 @@
   <transmission name="arm_trans">
     <type>transmission_interface/SimpleTransmission</type>
-    <joint name="arm_s_joint">
+    <joint name="arm_joint">
       <hardwareInterface>EffortJointInterface</hardwareInterface>
     </joint>
